Commit message: Added ahman_robot_arm_descp

File: robot_description/urdf/robot_arm.urdf.xacro (robot description, xacro)
@@ -4,4 +4,5 @@
      For more information, please see http://wiki.ros.org/sw_urdf_exporter -->
 <robot xmlns:xacro="http://ros.org/wiki/xacro" name="robot_description">
+  <xacro:include filename="$(find gripper_description)/urdf/gripper.urdf.xacro" />
   <link name="world_link"/>
 	<joint name="world_to_base_link=" type="fixed">
@@ -224,5 +225,5 @@
       velocity="0" />
   </joint>
-  <link
+  <!-- <link
     name="wrist_link">
     <inertial>
@@ -263,5 +264,5 @@
       </geometry>
     </collision>
-  </link>
+  </link> -->
   <joint
     name="wrist_joint"
@@ -273,5 +274,5 @@
       link="elbow_link" />
     <child
-      link="wrist_link" />
+      link="gripper_base_link" />
     <axis
       xyz="0 0 1" />
@@ -282,5 +283,5 @@
       velocity="0" />
   </joint>
-  <link
+  <!-- <link
     name="gripper_link">
     <inertial>
@@ -321,6 +322,6 @@
       </geometry>
     </collision>
-  </link>
-  <joint
+  </link> -->
+  <!-- <joint
     name="gripper_joint"
     type="revolute">
@@ -339,4 +340,4 @@
       effort="0"
       velocity="0" />
-  </joint>
+  </joint> -->
 </robot>
